Commit message: helm control configured

File: race_description/urdf/base.urdf.xacro (robot description, xacro)
@@ -3,5 +3,5 @@
     <link name="base_link">
         <visual>
-            <origin xyz="-0.2 0.0 0.0" rpy="1.5707 0.0 1.5707"/>
+            <origin xyz="0.456 0.0 0.0" rpy="3.1415926 0.0 0.0"/>
             <geometry>
                 <mesh filename="package://race_description/mesh/RACE_body.obj" scale="0.001 0.001 0.001"/>
@@ -11,5 +11,5 @@
     <link name="cg_link"/>
     <joint name="cg_joint" type="fixed">
-        <origin xyz="0.0 0.0 0.0" rpy="3.1415926 0.0 0.0"/>
+        <origin xyz="0.05 0.0 0.0" rpy="3.1415926 0.0 0.0"/>
         <parent link="base_link"/>
         <child link="cg_link"/>
@@ -17,5 +17,5 @@
     <link name="imu"/>
     <joint name="imu_joint" type="fixed">
-        <origin xyz="0.0 -0.09 0.0" rpy="3.1415926 0.0 0.0"/>
+        <origin xyz="0.05 0.0 0.1" rpy="3.1415926 0.0 0.0"/>
         <parent link="base_link"/>
         <child link="imu"/>
@@ -29,5 +29,5 @@
     <link name="dvl"/>
     <joint name="dvl_joint" type="fixed">
-        <origin xyz="0.0625 0.0 -0.1" rpy="3.1415926 0.0 0.0"/>
+        <origin xyz="-0.05 0.0 0.0" rpy="3.1415926 0.0 0.0"/>
         <parent link="base_link"/>
         <child link="dvl"/>
@@ -35,5 +35,5 @@
      <link name="dvl_sf"/>
     <joint name="dvl_sf_joint" type="fixed">
-        <origin xyz="-0.22 0.0 -0.08" rpy="0.0 0.0 0.0"/>
+        <origin xyz="-0.05 0.0 0.0" rpy="0.0 0.0 0.0"/>
         <parent link="base_link"/>
         <child link="dvl_sf"/>
@@ -41,5 +41,5 @@
     <link name="gps"/>
     <joint name="gps_joint" type="fixed">
-        <origin xyz="0.45 0.0 0.28" rpy="3.1415926 0.0 0.0"/>
+        <origin xyz="-0.05 0.0 0.18" rpy="0.0 0.0 0.0"/>
         <parent link="base_link"/>
         <child link="gps"/>
@@ -47,38 +47,44 @@
     <link name="pressure"/>
     <joint name="pressure_joint" type="fixed">
-        <origin xyz="0.32 0.0 0.05" rpy="3.1415926 0.0 0.0"/>
+        <origin xyz="-0.05 0.0 0.0" rpy="3.1415926 0.0 0.0"/>
         <parent link="base_link"/>
         <child link="pressure"/>
     </joint>
-    <link name="ping360_link"/>
-    <joint name="ping360_joint" type="fixed">
-        <origin xyz="0.592 0.0 -0.085" rpy="3.1415926 0.0 3.1415926"/>
+    <!-- thrusters -->
+    <link name="sway_stern_thruster_link"/>
+    <joint name="sway_stern_thruster_joint" type="fixed">
+        <origin xyz="-0.2075 0.0 0.07535" rpy="3.1415926 0.0 -1.571"/>
         <parent link="base_link"/>
-        <child link="ping360_link"/>
-    </joint>
-    <!-- thrusters -->
-    <link name="surge_thruster_link"/>
-    <joint name="surge_thruster_joint" type="fixed">
-        <origin xyz="-0.77 0.0 0.0" rpy="0.0 0.0 0.0"/>
-        <parent link="base_link"/>
-        <child link="surge_thruster_link"/>
+        <child link="sway_stern_thruster_link"/>
     </joint>
     <link name="heave_bow_thruster_link"/>
     <joint name="heave_bow_thruster_joint" type="fixed">
-        <origin xyz="0.387 0.0 0.0" rpy="0.0 -1.57079632679 0.0"/>
+        <origin xyz="0.38065 0.0 0.07535" rpy="3.1415926 -1.571 0.0"/>
         <parent link="base_link"/>
         <child link="heave_bow_thruster_link"/>
     </joint>
-    <link name="heave_stern_thruster_link"/>
-    <joint name="heave_stern_thruster_joint" type="fixed">
-        <origin xyz="-0.387 0.0 0.0" rpy="0.0 -1.57079632679 0.0"/>
+    <link name="heave_stern_port_thruster_link"/>
+    <joint name="heave_stern_port_thruster_joint" type="fixed">
+        <origin xyz="-0.104 -0.1034 0.07535" rpy="-1.571 -1.571 0.0"/>
         <parent link="base_link"/>
-        <child link="heave_stern_thruster_link"/>
+        <child link="heave_stern_port_thruster_link"/>
     </joint>
-    <link name="sway_bow_thruster_link"/>
-    <joint name="sway_bow_thruster_joint" type="fixed">
-        <origin xyz="0.51 0.0 0.0" rpy="0.0 0.0 1.57079632679"/>
+    <link name="heave_stern_stdb_thruster_link"/>
+    <joint name="heave_stern_stdb_thruster_joint" type="fixed">
+        <origin xyz="-0.104 0.1034 0.07535" rpy="1.571 -1.571 0.0"/>
         <parent link="base_link"/>
-        <child link="sway_bow_thruster_link"/>
+        <child link="heave_stern_stdb_thruster_link"/>
+    </joint>
+    <link name="surge_port_thruster_link"/>
+    <joint name="surge_port_thruster_joint" type="fixed">
+        <origin xyz="-0.404 0.125 0.05485" rpy="1.571 0.0 0.52"/>
+        <parent link="base_link"/>
+        <child link="surge_port_thruster_link"/>
+    </joint>
+    <link name="surge_stdb_thruster_link"/>
+    <joint name="surge_stdb_thruster_joint" type="fixed">
+        <origin xyz="-0.404 -0.125 0.05485" rpy="-1.571 0.0 -0.52"/>
+        <parent link="base_link"/>
+        <child link="surge_stdb_thruster_link"/>
     </joint>
 </robot>

Commit message: race auv test with rotated surge thruster

File: race_description/urdf/base.urdf.xacro (robot description, xacro)
@@ -11,5 +11,5 @@
     <link name="cg_link"/>
     <joint name="cg_joint" type="fixed">
-        <origin xyz="0.05 0.0 0.0" rpy="3.1415926 0.0 0.0"/>
+        <origin xyz="0.1 0.0 0.0" rpy="3.1415926 0.0 0.0"/>
         <parent link="base_link"/>
         <child link="cg_link"/>
@@ -60,5 +60,5 @@
     <link name="heave_bow_thruster_link"/>
     <joint name="heave_bow_thruster_joint" type="fixed">
-        <origin xyz="0.38065 0.0 0.07535" rpy="3.1415926 -1.571 0.0"/>
+        <origin xyz="0.38065 0.0 0.07535" rpy="3.1415926 1.571 0.0"/>
         <parent link="base_link"/>
         <child link="heave_bow_thruster_link"/>
@@ -66,5 +66,5 @@
     <link name="heave_stern_port_thruster_link"/>
     <joint name="heave_stern_port_thruster_joint" type="fixed">
-        <origin xyz="-0.104 -0.1034 0.07535" rpy="-1.571 -1.571 0.0"/>
+        <origin xyz="-0.104 -0.1034 0.07535" rpy="-1.571 1.571 0.0"/>
         <parent link="base_link"/>
         <child link="heave_stern_port_thruster_link"/>
@@ -72,5 +72,5 @@
     <link name="heave_stern_stdb_thruster_link"/>
     <joint name="heave_stern_stdb_thruster_joint" type="fixed">
-        <origin xyz="-0.104 0.1034 0.07535" rpy="1.571 -1.571 0.0"/>
+        <origin xyz="-0.104 0.1034 0.07535" rpy="1.571 1.571 0.0"/>
         <parent link="base_link"/>
         <child link="heave_stern_stdb_thruster_link"/>
@@ -78,5 +78,5 @@
     <link name="surge_port_thruster_link"/>
     <joint name="surge_port_thruster_joint" type="fixed">
-        <origin xyz="-0.404 0.125 0.05485" rpy="1.571 0.0 0.52"/>
+        <origin xyz="-0.404 0.125 0.05485" rpy="1.571 -0.8 0.52"/>
         <parent link="base_link"/>
         <child link="surge_port_thruster_link"/>
@@ -84,5 +84,5 @@
     <link name="surge_stdb_thruster_link"/>
     <joint name="surge_stdb_thruster_joint" type="fixed">
-        <origin xyz="-0.404 -0.125 0.05485" rpy="-1.571 0.0 -0.52"/>
+        <origin xyz="-0.404 -0.125 0.05485" rpy="-1.571 -0.8 -0.52"/>
         <parent link="base_link"/>
         <child link="surge_stdb_thruster_link"/>

Commit message: race config updated

File: race_description/urdf/base.urdf.xacro (robot description, xacro)
@@ -78,5 +78,5 @@
     <link name="surge_port_thruster_link"/>
     <joint name="surge_port_thruster_joint" type="fixed">
-        <origin xyz="-0.404 0.125 0.05485" rpy="1.571 -0.8 0.52"/>
+        <origin xyz="-0.404 0.125 0.05485" rpy="1.571 0.0 0.52"/>
         <parent link="base_link"/>
         <child link="surge_port_thruster_link"/>
@@ -84,5 +84,5 @@
     <link name="surge_stdb_thruster_link"/>
     <joint name="surge_stdb_thruster_joint" type="fixed">
-        <origin xyz="-0.404 -0.125 0.05485" rpy="-1.571 -0.8 -0.52"/>
+        <origin xyz="-0.404 -0.125 0.05485" rpy="-1.571 0.0 -0.52"/>
         <parent link="base_link"/>
         <child link="surge_stdb_thruster_link"/>

Commit message: adjusted urdf

File: race_description/urdf/base.urdf.xacro (robot description, xacro)
@@ -11,5 +11,5 @@
     <link name="cg_link"/>
     <joint name="cg_joint" type="fixed">
-        <origin xyz="0.1 0.0 0.0" rpy="3.1415926 0.0 0.0"/>
+        <origin xyz="0.0 0.0 0.0" rpy="3.1415926 0.0 0.0"/>
         <parent link="base_link"/>
         <child link="cg_link"/>
@@ -17,5 +17,5 @@
     <link name="imu"/>
     <joint name="imu_joint" type="fixed">
-        <origin xyz="0.05 0.0 0.1" rpy="3.1415926 0.0 0.0"/>
+        <origin xyz="-0.05 0.0 0.05" rpy="3.1415926 0.0 0.0"/>
         <parent link="base_link"/>
         <child link="imu"/>
@@ -29,5 +29,5 @@
     <link name="dvl"/>
     <joint name="dvl_joint" type="fixed">
-        <origin xyz="-0.05 0.0 0.0" rpy="3.1415926 0.0 0.0"/>
+        <origin xyz="0.0 0.0 -0.09" rpy="3.1415926 0.0 0.0"/>
         <parent link="base_link"/>
         <child link="dvl"/>
@@ -35,5 +35,5 @@
      <link name="dvl_sf"/>
     <joint name="dvl_sf_joint" type="fixed">
-        <origin xyz="-0.05 0.0 0.0" rpy="0.0 0.0 0.0"/>
+        <origin xyz="-0.00 0.0 -0.09" rpy="0.0 0.0 0.0"/>
         <parent link="base_link"/>
         <child link="dvl_sf"/>
@@ -41,5 +41,5 @@
     <link name="gps"/>
     <joint name="gps_joint" type="fixed">
-        <origin xyz="-0.05 0.0 0.18" rpy="0.0 0.0 0.0"/>
+        <origin xyz="0.25 0.1 0.4" rpy="0.0 0.0 0.0"/>
         <parent link="base_link"/>
         <child link="gps"/>
@@ -47,5 +47,5 @@
     <link name="pressure"/>
     <joint name="pressure_joint" type="fixed">
-        <origin xyz="-0.05 0.0 0.0" rpy="3.1415926 0.0 0.0"/>
+        <origin xyz="0.1 0.0 0.0" rpy="3.1415926 0.0 0.0"/>
         <parent link="base_link"/>
         <child link="pressure"/>

Commit message: updated config for race test

File: race_description/urdf/base.urdf.xacro (robot description, xacro)
@@ -33,5 +33,5 @@
         <child link="dvl"/>
     </joint>
-     <link name="dvl_sf"/>
+    <link name="dvl_sf"/>
     <joint name="dvl_sf_joint" type="fixed">
         <origin xyz="-0.00 0.0 -0.09" rpy="0.0 0.0 0.0"/>

Commit message: fixed small issue in launch files

File: race_description/urdf/base.urdf.xacro (robot description, xacro)
@@ -17,5 +17,5 @@
     <link name="imu"/>
     <joint name="imu_joint" type="fixed">
-        <origin xyz="-0.05 0.0 0.05" rpy="3.1415926 0.0 0.0"/>
+        <origin xyz="-0.05 0.0 0.15" rpy="3.1415926 0.0 0.0"/>
         <parent link="base_link"/>
         <child link="imu"/>

Commit message: fixed thruster urdf and teleop ymal

File: race_description/urdf/base.urdf.xacro (robot description, xacro)
@@ -66,5 +66,5 @@
     <link name="heave_stern_port_thruster_link"/>
     <joint name="heave_stern_port_thruster_joint" type="fixed">
-        <origin xyz="-0.104 -0.1034 0.07535" rpy="-1.571 1.571 0.0"/>
+        <origin xyz="-0.104 0.1034 0.07535" rpy="-1.571 1.571 0.0"/>
         <parent link="base_link"/>
         <child link="heave_stern_port_thruster_link"/>
@@ -72,5 +72,5 @@
     <link name="heave_stern_stdb_thruster_link"/>
     <joint name="heave_stern_stdb_thruster_joint" type="fixed">
-        <origin xyz="-0.104 0.1034 0.07535" rpy="1.571 1.571 0.0"/>
+        <origin xyz="-0.104 -0.1034 0.07535" rpy="1.571 1.571 0.0"/>
         <parent link="base_link"/>
         <child link="heave_stern_stdb_thruster_link"/>

Commit message: new microstrain driver

File: race_description/urdf/base.urdf.xacro (robot description, xacro)
@@ -17,5 +17,6 @@
     <link name="imu"/>
     <joint name="imu_joint" type="fixed">
-        <origin xyz="-0.05 0.0 0.15" rpy="3.1415926 0.0 0.0"/>
+        <!-- <origin xyz="-0.05 0.0 0.15" rpy="3.1415926 0.0 0.0"/> -->
+        <origin xyz="-0.05 0.0 0.15" rpy="0.0 0.0 0.0"/>
         <parent link="base_link"/>
         <child link="imu"/>

Commit message: Update base.urdf.xacro

File: race_description/urdf/base.urdf.xacro (robot description, xacro)
@@ -18,5 +18,5 @@
     <joint name="imu_joint" type="fixed">
         <!-- <origin xyz="-0.05 0.0 0.15" rpy="3.1415926 0.0 0.0"/> -->
-        <origin xyz="-0.05 0.0 0.15" rpy="0.0 0.0 0.0"/>
+        <origin xyz="0.0 0.0 0.12" rpy="0.0 0.0 0.0"/>
         <parent link="base_link"/>
         <child link="imu"/>
@@ -42,5 +42,5 @@
     <link name="gps"/>
     <joint name="gps_joint" type="fixed">
-        <origin xyz="0.25 0.1 0.4" rpy="0.0 0.0 0.0"/>
+        <origin xyz="0.22 -0.1 0.4" rpy="0.0 0.0 0.0"/>
         <parent link="base_link"/>
         <child link="gps"/>
@@ -48,5 +48,5 @@
     <link name="pressure"/>
     <joint name="pressure_joint" type="fixed">
-        <origin xyz="0.1 0.0 0.0" rpy="3.1415926 0.0 0.0"/>
+        <origin xyz="0.2 0.0 -0.09" rpy="3.1415926 0.0 0.0"/>
         <parent link="base_link"/>
         <child link="pressure"/>
@@ -55,5 +55,5 @@
     <link name="sway_stern_thruster_link"/>
     <joint name="sway_stern_thruster_joint" type="fixed">
-        <origin xyz="-0.2075 0.0 0.07535" rpy="3.1415926 0.0 -1.571"/>
+        <origin xyz="-0.29 0.0 0.07535" rpy="3.1415926 0.0 -1.571"/>
         <parent link="base_link"/>
         <child link="sway_stern_thruster_link"/>
@@ -61,5 +61,5 @@
     <link name="heave_bow_thruster_link"/>
     <joint name="heave_bow_thruster_joint" type="fixed">
-        <origin xyz="0.38065 0.0 0.07535" rpy="3.1415926 1.571 0.0"/>
+        <origin xyz="0.3 0.0 0.07535" rpy="3.1415926 1.571 0.0"/>
         <parent link="base_link"/>
         <child link="heave_bow_thruster_link"/>
@@ -67,5 +67,5 @@
     <link name="heave_stern_port_thruster_link"/>
     <joint name="heave_stern_port_thruster_joint" type="fixed">
-        <origin xyz="-0.104 0.1034 0.07535" rpy="-1.571 1.571 0.0"/>
+        <origin xyz="-0.19 0.1034 0.07535" rpy="-1.571 1.571 0.0"/>
         <parent link="base_link"/>
         <child link="heave_stern_port_thruster_link"/>
@@ -73,5 +73,5 @@
     <link name="heave_stern_stdb_thruster_link"/>
     <joint name="heave_stern_stdb_thruster_joint" type="fixed">
-        <origin xyz="-0.104 -0.1034 0.07535" rpy="1.571 1.571 0.0"/>
+        <origin xyz="-0.19 -0.1034 0.07535" rpy="1.571 1.571 0.0"/>
         <parent link="base_link"/>
         <child link="heave_stern_stdb_thruster_link"/>
@@ -79,5 +79,5 @@
     <link name="surge_port_thruster_link"/>
     <joint name="surge_port_thruster_joint" type="fixed">
-        <origin xyz="-0.404 0.125 0.05485" rpy="1.571 0.0 0.52"/>
+        <origin xyz="-0.41 0.125 0.05485" rpy="1.571 0.0 0.52"/>
         <parent link="base_link"/>
         <child link="surge_port_thruster_link"/>
@@ -85,5 +85,5 @@
     <link name="surge_stdb_thruster_link"/>
     <joint name="surge_stdb_thruster_joint" type="fixed">
-        <origin xyz="-0.404 -0.125 0.05485" rpy="-1.571 0.0 -0.52"/>
+        <origin xyz="-0.41 -0.125 0.05485" rpy="-1.571 0.0 -0.52"/>
         <parent link="base_link"/>
         <child link="surge_stdb_thruster_link"/>

Commit message: camera_urdf

File: race_description/urdf/base.urdf.xacro (robot description, xacro)
@@ -52,4 +52,10 @@
         <child link="pressure"/>
     </joint>
+    <link name="camera"/>
+    <joint name="camera_joint" type="fixed">
+        <origin xyz="0.3 0.23 -0.05" rpy="3.1415926 0.0 0.0"/>
+        <parent link="base_link"/>
+        <child link="camera"/>
+    </joint>
     <!-- thrusters -->
     <link name="sway_stern_thruster_link"/>

Commit message: updated urdf

File: race_description/urdf/base.urdf.xacro (robot description, xacro)
@@ -61,5 +61,5 @@
     <link name="sway_stern_thruster_link"/>
     <joint name="sway_stern_thruster_joint" type="fixed">
-        <origin xyz="-0.29 0.0 0.07535" rpy="3.1415926 0.0 -1.571"/>
+        <origin xyz="-0.29 0.0 -0.07535" rpy="3.1415926 0.0 -1.571"/>
         <parent link="base_link"/>
         <child link="sway_stern_thruster_link"/>
@@ -67,5 +67,5 @@
     <link name="heave_bow_thruster_link"/>
     <joint name="heave_bow_thruster_joint" type="fixed">
-        <origin xyz="0.3 0.0 0.07535" rpy="3.1415926 1.571 0.0"/>
+        <origin xyz="0.3 0.0 -0.07535" rpy="3.1415926 1.571 0.0"/>
         <parent link="base_link"/>
         <child link="heave_bow_thruster_link"/>
@@ -73,5 +73,5 @@
     <link name="heave_stern_port_thruster_link"/>
     <joint name="heave_stern_port_thruster_joint" type="fixed">
-        <origin xyz="-0.19 0.1034 0.07535" rpy="-1.571 1.571 0.0"/>
+        <origin xyz="-0.19 0.1034 -0.07535" rpy="-1.571 1.571 0.0"/>
         <parent link="base_link"/>
         <child link="heave_stern_port_thruster_link"/>
@@ -79,5 +79,5 @@
     <link name="heave_stern_stdb_thruster_link"/>
     <joint name="heave_stern_stdb_thruster_joint" type="fixed">
-        <origin xyz="-0.19 -0.1034 0.07535" rpy="1.571 1.571 0.0"/>
+        <origin xyz="-0.19 -0.1034 -0.07535" rpy="1.571 1.571 0.0"/>
         <parent link="base_link"/>
         <child link="heave_stern_stdb_thruster_link"/>
@@ -85,5 +85,5 @@
     <link name="surge_port_thruster_link"/>
     <joint name="surge_port_thruster_joint" type="fixed">
-        <origin xyz="-0.41 0.125 0.05485" rpy="1.571 0.0 0.52"/>
+        <origin xyz="-0.41 0.125 -0.10" rpy="1.571 0.0 0.52"/>
         <parent link="base_link"/>
         <child link="surge_port_thruster_link"/>
@@ -91,5 +91,5 @@
     <link name="surge_stdb_thruster_link"/>
     <joint name="surge_stdb_thruster_joint" type="fixed">
-        <origin xyz="-0.41 -0.125 0.05485" rpy="-1.571 0.0 -0.52"/>
+        <origin xyz="-0.41 -0.125 -0.10" rpy="-1.571 0.0 -0.52"/>
         <parent link="base_link"/>
         <child link="surge_stdb_thruster_link"/>

Commit message: allen harbor pid tunning

File: race_description/urdf/base.urdf.xacro (robot description, xacro)
@@ -61,4 +61,5 @@
     <link name="sway_stern_thruster_link"/>
     <joint name="sway_stern_thruster_joint" type="fixed">
+        <!-- <origin xyz="-0.29 0.0 -0.07535" rpy="3.1415926 0.0 -1.571"/> -->
         <origin xyz="-0.29 0.0 -0.07535" rpy="3.1415926 0.0 -1.571"/>
         <parent link="base_link"/>
@@ -85,5 +86,6 @@
     <link name="surge_port_thruster_link"/>
     <joint name="surge_port_thruster_joint" type="fixed">
-        <origin xyz="-0.41 0.125 -0.10" rpy="1.571 0.0 0.52"/>
+        <!-- <origin xyz="-0.41 0.125 -0.10" rpy="1.571 0.0 0.52"/> -->
+        <origin xyz="-0.41 0.125 0.01" rpy="1.571 0.0 0.52"/>
         <parent link="base_link"/>
         <child link="surge_port_thruster_link"/>
@@ -91,5 +93,6 @@
     <link name="surge_stdb_thruster_link"/>
     <joint name="surge_stdb_thruster_joint" type="fixed">
-        <origin xyz="-0.41 -0.125 -0.10" rpy="-1.571 0.0 -0.52"/>
+        <!-- <origin xyz="-0.41 -0.125 -0.10" rpy="-1.571 0.0 -0.52"/> -->
+        <origin xyz="-0.41 -0.125 0.01" rpy="-1.571 0.0 -0.52"/>
         <parent link="base_link"/>
         <child link="surge_stdb_thruster_link"/>
