Commit message: building stonefish simulation launch and config files

File: race_auv_description/urdf/base.urdf (robot description, URDF)
Before this commit: robot race_auv, 15 links, 14 joints
Links:
- added link cam
Joints:
- added joint cam_joint: type fixed, parent nose_tip_link, child cam, origin xyz=0.0 0.0 0.0 rpy=0.0 0.0 0.0

Commit message: basic simulation working

File: race_auv_description/urdf/base.urdf (robot description, URDF)
Before this commit: robot race_auv, 16 links, 15 joints
Joints:
- joint surge_port_thruster_joint: origin xyz=-0.86 -0.125 -0.05485 rpy=0.0 0.8 -0.52 -> xyz=-0.875 -0.11 -0.05485 rpy=0.0 0.0 -0.52
- joint surge_stbd_thruster_joint: origin xyz=-0.86 0.125 -0.05485 rpy=0.0 0.8 0.52 -> xyz=-0.875 0.11 -0.05485 rpy=0.0 0.0 0.52

Commit message: two cam

File: race_auv_description/urdf/base.urdf (robot description, URDF)
Before this commit: robot race_auv, 16 links, 15 joints
Links:
- removed link cam
- added link cam1
- added link cam2
Joints:
- removed joint cam_joint
- added joint cam1_joint: type fixed, parent nose_tip_link, child cam1, origin xyz=0.0 0.0 0.0 rpy=0.0 0.0 0.0
- added joint cam2_joint: type fixed, parent nose_tip_link, child cam2, origin xyz=0.0 0.0 0.0 rpy=0.0 0.0 0.0

Commit message: apriltag detection

File: race_auv_description/urdf/base.urdf (robot description, URDF)
Before this commit: robot race_auv, 17 links, 16 joints
Joints:
- joint cam1_joint: origin xyz=0.0 0.0 0.0 rpy=0.0 0.0 0.0 -> xyz=0.0 0.0 -0.05 rpy=1.571 0.0 1.571; parent nose_tip_link -> base_link
- joint cam2_joint: parent nose_tip_link -> base_link

Commit message: new apriltag detection & tag/station tf pub

File: race_auv_description/urdf/base.urdf (robot description, URDF)
Before this commit: robot race_auv, 17 links, 16 joints
Joints:
- joint cam2_joint: origin xyz=0.0 0.0 0.0 rpy=0.0 0.0 0.0 -> xyz=-0.3 0.0 0.01 rpy=0.0 0.0 1.571
