Commit message: updated docking sim

File: race_auv_description/urdf/base.urdf (robot description, URDF)
Before this commit: robot race_auv, 17 links, 16 joints
Links:
- removed link cam1
- removed link cam2
- removed link gps
- added link acomm_modem
- added link cam_down
- added link cam_front
Joints:
- removed joint cam1_joint
- removed joint cam2_joint
- removed joint gps_joint
- added joint acomm_modem_joint: type fixed, parent nose_tip_link, child acomm_modem, origin xyz=-0.268 0.1 0.095 rpy=0.0 0.0 0.0
- added joint cam_down_joint: type fixed, parent nose_tip_link, child cam_down, origin xyz=-0.305 0.0 -0.153 rpy=0.0 3.1415 1.571
- added joint cam_front_joint: type fixed, parent nose_tip_link, child cam_front, origin xyz=-0.004 0.0 0.035 rpy=-1.571 0.0 -1.571
- joint base_link: origin xyz=0.0 0.0 0.0 rpy=0.0 0.0 0.0 -> xyz=0.6 0.0 0.0 rpy=0.0 0.0 0.0
- joint dvl_joint: origin xyz=-0.5 0.0 0.0 rpy=3.1415926 0.0 0.0 -> xyz=-0.738 0.0 -0.138 rpy=3.1415926 0.0 0.0; parent base_link -> nose_tip_link
- joint dvl_sf_joint: origin xyz=-0.5 0.0 0.0 rpy=3.1415926 0.0 0.0 -> xyz=-0.738 0.0 -0.138 rpy=0.0 0.0 0.0; parent base_link -> nose_tip_link
- joint heave_bow_thruster_joint: origin xyz=-0.07535 0.0 -0.07535 rpy=0.0 -1.571 0.0 -> xyz=-0.186 0.0 -0.016 rpy=0.0 -1.571 0.0; parent base_link -> nose_tip_link
- joint heave_stern_port_thruster_joint: origin xyz=-0.56 -0.1034 -0.07535 rpy=0.0 -1.571 0.0 -> xyz=-0.928 0.103 -0.016 rpy=0.0 -1.571 0.0; parent base_link -> nose_tip_link
- joint heave_stern_stbd_thruster_joint: origin xyz=-0.56 0.1034 -0.07535 rpy=0.0 -1.571 0.0 -> xyz=-0.928 -0.103 -0.016 rpy=0.0 -1.571 0.0; parent base_link -> nose_tip_link
- joint imu__sf_joint: origin xyz=-0.5 0.0 -0.08 rpy=0.0 0.0 0.0 -> xyz=-0.621 0.0 -0.120 rpy=0.0 0.0 0.0; parent base_link -> nose_tip_link
- joint imu_joint: origin xyz=-0.5 0.0 -0.08 rpy=0.0 0.0 0.0 -> xyz=-0.621 0.0 -0.120 rpy=0.0 0.0 0.0; parent base_link -> nose_tip_link
- joint pressure_joint: origin xyz=-0.2 0.0 0.0 rpy=0.0 0.0 0.0 -> xyz=-0.524 0 -0.021 rpy=0.0 0.0 0.0; parent base_link -> nose_tip_link
- joint surge_port_thruster_joint: origin xyz=-0.875 -0.11 -0.05485 rpy=0.0 0.0 -0.52 -> xyz=-1.273 0.09 -0.03 rpy=0.0 0.0 0.52; parent base_link -> nose_tip_link
- joint surge_stbd_thruster_joint: origin xyz=-0.875 0.11 -0.05485 rpy=0.0 0.0 0.52 -> xyz=-1.273 -0.09 -0.03 rpy=0.0 0.0 -0.52; parent base_link -> nose_tip_link
- joint sway_stern_thruster_joint: origin xyz=-0.66635 0.0 -0.07535 rpy=0.0 0.0 1.571 -> xyz=-1.043 -0.005 -0.011 rpy=0.0 0.0 1.571; parent base_link -> nose_tip_link

Commit message: race auv dock point tf

File: race_auv_description/urdf/base.urdf (robot description, URDF)
Before this commit: robot race_auv, 17 links, 16 joints
Links:
- added link auv_dock_point_link
Joints:
- added joint auv_dock_point_joint: type fixed, parent nose_tip_link, child auv_dock_point_link, origin xyz=-0.305 0.0 -0.13 rpy=0.0 0.0 0.0
- joint cam_down_joint: origin xyz=-0.305 0.0 -0.153 rpy=0.0 3.1415 1.571 -> xyz=-0.305 0.0 -0.128 rpy=0.0 3.1415 1.571

Commit message: race auv dock point tf rename

File: race_auv_description/urdf/base.urdf (robot description, URDF)
Before this commit: robot race_auv, 18 links, 17 joints
Links:
- removed link auv_dock_point_link
- added link auv_dock_point
Joints:
- joint auv_dock_point_joint: child auv_dock_point_link -> auv_dock_point

Commit message: updated urdf heave x and imu, mcu installed true

File: race_auv_description/urdf/base.urdf (robot description, URDF)
Before this commit: robot race_auv, 18 links, 17 joints
Joints:
- joint heave_bow_thruster_joint: origin xyz=-0.186 0.0 -0.016 rpy=0.0 -1.571 0.0 -> xyz=-0.186 0.0 -0.016 rpy=0.0 1.571 0.0
- joint heave_stern_port_thruster_joint: origin xyz=-0.928 0.103 -0.016 rpy=0.0 -1.571 0.0 -> xyz=-0.928 0.103 -0.016 rpy=0.0 1.571 0.0
- joint heave_stern_stbd_thruster_joint: origin xyz=-0.928 -0.103 -0.016 rpy=0.0 -1.571 0.0 -> xyz=-0.928 -0.103 -0.016 rpy=0.0 1.571 0.0
- joint imu_joint: origin xyz=-0.621 0.0 -0.120 rpy=0.0 0.0 0.0 -> xyz=-0.621 0.0 -0.120 rpy=3.1415926 0.0 3.1415926

Commit message: after tank test aug1826

File: race_auv_description/urdf/base.urdf (robot description, URDF)
Before this commit: robot race_auv, 18 links, 17 joints
Joints:
- joint imu_joint: origin xyz=-0.621 0.0 -0.120 rpy=3.1415926 0.0 3.1415926 -> xyz=-0.621 0.0 -0.120 rpy=0.0 0.0 -3.1415926

Commit message: updated configs and t200 polynomials

File: race_auv_description/urdf/base.urdf (robot description, URDF)
Before this commit: robot race_auv, 18 links, 17 joints
Joints:
- joint base_link: origin xyz=0.6 0.0 0.0 rpy=0.0 0.0 0.0 -> xyz=0.7 0.0 0.0 rpy=0.0 0.0 0.0
- joint surge_port_thruster_joint: origin xyz=-1.273 0.09 -0.03 rpy=0.0 0.0 0.52 -> xyz=-1.273 0.09 -0.03 rpy=0.0 0.0 0.53

Commit message: update from past tank test

File: race_auv_description/urdf/base.urdf (robot description, URDF)
Before this commit: robot race_auv, 18 links, 17 joints
Links:
- added link cb_link
Joints:
- added joint cb_joint: type fixed, parent base_link, child cb_link, origin xyz=0.0 0.0 0.05 rpy=0.0 0.0 0.0
